File: Kicad1/kicad1.kicad_sch (KiCad schematic)
At the start: 37 parts, among them J1 M1_CONN, J2 M1_CONN, J3 BATT_CONN, J4 Conn_01x08, J5 ESP_CONN, J6 ENCODER_CONN, J7 Conn_01x04, J8 USB_C_Receptacle_USB2.0_14P, U1 STM32F401RBTx, U2 LD1117S50TR_SOT223, U3 LD1117S33TR_SOT223, U4 TB6612FNG, Y1 Crystal_GND24

Commit message: Add files via upload
Parts:
- added C17: 10 µF, Capacitor_Tantalum_SMD:CP_EIA-6032-28_Kemet-C_HandSolder, symbol Device:C_Polarized_Small_US
- added C18, C19, C21: 0.1 µF, Capacitor_SMD:C_0805_2012Metric_Pad1.18x1.45mm_HandSolder, symbol Device:C_Small
- added C20: 0.01 µF, Capacitor_SMD:C_0805_2012Metric_Pad1.18x1.45mm_HandSolder, symbol Device:C_Small
- added C22: 2.2 µF, Capacitor_SMD:C_0805_2012Metric_Pad1.18x1.45mm_HandSolder, symbol Device:C_Small
- added D3: WS2812B, LED_SMD:LED_WS2812B_PLCC4_5.0x5.0mm_P3.2mm, symbol LED:WS2812B
- added D4: USB_LED, LED_SMD:LED_0805_2012Metric_Pad1.15x1.40mm_HandSolder, symbol Device:LED
- added D5: USER_LED, LED_SMD:LED_0805_2012Metric_Pad1.15x1.40mm_HandSolder, symbol Device:LED
- added F1: PTCSMD, Fuse:Fuse_1812_4532Metric, symbol Device:Polyfuse_Small
- added J9: MT6701_CONN, Connector_JST:JST_XH_B5B-XH-A_1x05_P2.50mm_Vertical, symbol Connector_Generic:Conn_01x05
- added R10, R9: 1 kΩ, Resistor_SMD:R_0805_2012Metric_Pad1.20x1.40mm_HandSolder, symbol Device:R
- added R5, R6: 5.1 kΩ, Resistor_SMD:R_0603_1608Metric_Pad0.98x0.95mm_HandSolder, symbol Device:R
- added R7, R8: 22 Ω, Resistor_SMD:R_0805_2012Metric_Pad1.20x1.40mm_HandSolder, symbol Device:R
- added SW1: SW_UP_Reset, SW_uP_Reset:SW_uP_Reset, symbol Switch:SW_DPST_x2
- added U5: USBLC6-2SC6, Package_TO_SOT_SMD:SOT-23-6, symbol Power_Protection:USBLC6-2SC6
- C1, C2: footprint Capacitor_SMD:C_0603_1608Metric -> Capacitor_SMD:C_0805_2012Metric_Pad1.18x1.45mm_HandSolder
- C10, C11, C12, C13, C14, C3, C4, C5, C6, C7, C8, C9: footprint (none) -> Capacitor_SMD:C_0805_2012Metric_Pad1.18x1.45mm_HandSolder
- C15, C16: value C_Small -> 22 pF; footprint (none) -> Capacitor_SMD:C_0805_2012Metric_Pad1.18x1.45mm_HandSolder
- D1: value LED -> 5V_LED; footprint LED_SMD:LED_0805_2012Metric -> LED_SMD:LED_0805_2012Metric_Pad1.15x1.40mm_HandSolder
- D2: value LED -> 3V3_LED; footprint (none) -> LED_SMD:LED_0805_2012Metric_Pad1.15x1.40mm_HandSolder
- J1, J3: footprint (none) -> Connector_JST:JST_XH_B2B-XH-A_1x02_P2.50mm_Vertical
- J2: value M1_CONN -> M2_CONN; footprint (none) -> Connector_JST:JST_XH_B2B-XH-A_1x02_P2.50mm_Vertical
- J4: value Conn_01x08 -> Conn_MPU6050; footprint (none) -> Connector_PinSocket_2.54mm:PinSocket_1x08_P2.54mm_Vertical
- J8: footprint (none) -> Connector_USB:USB_C_Receptacle_HCTL_HC-TYPE-C-16P-01A
- R1, R2: value 1kΩ -> 1 kΩ; footprint (none) -> Resistor_SMD:R_0805_2012Metric_Pad1.20x1.40mm_HandSolder
- R3: value R -> 10K; footprint (none) -> Resistor_SMD:R_0805_2012Metric_Pad1.20x1.40mm_HandSolder
- R4: value R -> 10k; footprint (none) -> Resistor_SMD:R_0805_2012Metric_Pad1.20x1.40mm_HandSolder
- S1: value SLW-66527511-SMT-TR -> RST_SWITCH
- S2: footprint SLW-66527511-SMT-TR:SW_SLW-66527511-SMT-TR -> SW_SLW-66527511-SMT-TR:SW_SLW-66527511-SMT-TR
- Y1: value Crystal_GND24 -> 16MHz
Connections:
- net MD_A01 is gone; now on net MD_AO1: J1.1 (Pin_1)
- net MD_A02 is gone; now on net MD_AO2: J1.2 (Pin_2)
- net MD_B01 is gone; now on net MD_BO1: J2.1 (Pin_1)
- net MD_B02 is gone; now on net MD_BO2: J2.2 (Pin_2)
- net SWDIN is gone; now on net SWDIO: J7.1 (Pin_1)
- net +3.3V: now also S1.3, U1.13 (VREF+), C21.2, J9.1 (Pin_1)
- net +5V: now also J4.1 (Pin_1), S2.2, C19.1, D3.1 (VDD); no longer S2.3
- net ENC_A: now also U1.59 (PB7)
- net ENC_B: now also U1.58 (PB6)
- net ESP_RX: now also U1.42 (PA9)
- net ESP_TX: now also U1.43 (PA10)
- net GND: now also J4.2 (Pin_2), J8.A1 (GND), J8.A12 (GND), J8.B1 (GND), J8.B12 (GND), J8.S1 (SHIELD), S1.1, U1.12 (VSSA), U1.18 (VSS), U1.28 (PB2), U1.31 (VSS), U1.47 (VSS), U1.63 (VSS), U4.10 (PGND2), U4.18 (GND), U4.3 (PGND1), U4.4 (PGND1), U4.9 (PGND2), C17.2, C18.2, C19.2, C20.2, C21.1, C22.2, D3.3 (VSS), D4.1 (K), D5.1 (K), J9.2 (Pin_2), R5.2, R6.1, SW1.1 (A), U5.2 (GND)
- net SWCLK: now also U1.49 (PA14)
- net VM: now also C17.1, C18.1
- net WS_DIN: now reaches U1.14 (PA0)
- net WS_DIN: now also D3.4 (DIN)
- net MD_PWMA: now reaches U1.15 (PA1)
- net MD_PWMA: now also U4.23 (PWMA)
- net MD_AIN2: now reaches U1.16 (PA2)
- net MD_AIN2: now also U4.22 (AIN2)
- net MD_AIN1: now reaches U1.17 (PA3)
- net MD_AIN1: now also U4.21 (AIN1)
- net IMU_INT: now reaches U1.2 (PC13)
- net IMU_INT: now also J4.8 (Pin_8)
- net MD_STBY: now reaches U1.20 (PA4)
- net MD_STBY: now also U4.19 (STBY)
- net MD_PWMB: now reaches U1.21 (PA5)
- net MD_PWMB: now also U4.15 (PWMB)
- net MD_BIN1: now reaches U1.22 (PA6)
- net MD_BIN1: now also U4.17 (BIN1)
- net MD_BIN2: now reaches U1.23 (PA7)
- net MD_BIN2: now also U4.16 (BIN2)
- net USER_LED: now reaches U1.27 (PB1)
- net USER_LED: now also R10.1
- net at U1.30 (VCAP1): now also C22.1
- net MT_PWM: now reaches U1.37 (PC6)
- net MT_PWM: now also J9.3 (Pin_3)
- net MT_SDA: now reaches U1.40 (PC9)
- net MT_SDA: now also J9.5 (Pin_5)
- net MT_SCL: now reaches U1.41 (PA8)
- net MT_SCL: now also J9.4 (Pin_4)
- net ESD_D-: now reaches U1.44 (PA11)
- net ESD_D-: now also R7.1
- net ESD_D+: now reaches U1.45 (PA12)
- net ESD_D+: now also R8.1
- net SWDIO: now reaches U1.46 (PA13)
- net IMU_SCL: now reaches U1.61 (PB8)
- net IMU_SCL: now also J4.3 (Pin_3)
- net IMU_SDA: now reaches U1.62 (PB9)
- net IMU_SDA: now also J4.4 (Pin_4)
- net at U1.7 (NRST): now also C20.1, SW1.2 (B)
- net MD_AO1: now reaches U4.1 (AO1), U4.2 (AO1)
- net MD_BO1: now reaches U4.11 (BO1), U4.12 (BO1)
- net MD_AO2: now reaches U4.5 (AO2), U4.6 (AO2)
- net MD_BO2: now reaches U4.7 (BO2), U4.8 (BO2)
- net at J8.A4 (VBUS), J8.A9 (VBUS), J8.B4 (VBUS)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: now also F1.1
- net at J8.A5 (CC1): now also R5.1
- net at J8.A6 (D+): now also J8.B6 (D+), U5.3 (I/O2)
- net at J8.A7 (D-): now also J8.B7 (D-), U5.1 (I/O1)
- net at J8.B5 (CC2): now also R6.2
- new net: D4.2 (A), R9.2
- new net: D5.2 (A), R10.2
- new net: R8.2, U5.4 (I/O2)
- new net: R7.2, U5.6 (I/O1)
- new net Vusb: F1.2, R9.1, S2.3, U5.5 (VBUS)
- no-connect marks 2 -> 31
Other:
- note added: "BOOTO"
- note added: "CONN_D+"
- note added: "CONN_D-"
- note added: "IMU (MPU6050)"
- note added: "MOTOR DRIVER"
- note added: "MT6701"
- note added: "OSCIN"
- note added: "OSCOUT"
- note added: "USB_D+"
- note added: "USB_D-"
- note added: "WS2812"
- moved on the sheet: C1, C10, C11, C12, C13, C15, C16, C2, C3, C4, C5, C6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
