File: BalanceRobot/Kicad1.kicad_pcb (KiCad board)
At the start: 2 copper layers, 56 parts, among them J1 M1_CONN, J2 M2_CONN, J3 BATT_CONN, J4 Conn_MPU6050, J5 ESP_CONN, J6 ENCODER_CONN, J7 Conn_01x04, J8 USB_C_Receptacle_USB2.0_14P, J9 MT6701_CONN, SW1 SW_UP_Reset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

Commit message: Add files via upload
Parts:
- moved C18 88.0 mm to (184.5, 105.0)
- moved C17 87.7 mm to (180.5, 104.4)
- moved C14 80.0 mm to (142.0, 114.5), turned to 0 degrees
- moved U4 74.6 mm to (133.5, 116.0)
- moved D3 72.3 mm to (110.1, 104.3)
- moved C19 69.3 mm to (108.5, 98.5)
- moved J7 68.0 mm to (154.9, 55.5)
- moved R3 65.8 mm to (169.0, 92.0), turned to 90 degrees
- moved J9 65.8 mm to (160.0, 101.5)
- moved J5 61.4 mm to (172.5, 95.6), turned to 180 degrees
- moved J2 59.6 mm to (122.1, 124.7), turned to 90 degrees
- moved J1 57.5 mm to (123.1, 112.9), turned to -90 degrees
- moved J6 49.6 mm to (151.0, 71.0)
- moved S2 43.5 mm to (182.0, 64.0), turned to -90 degrees
- moved J3 40.4 mm to (172.0, 43.5)
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Connections:
- C15 pad 1: GND -> Net-(U1-PH0)
- J1 pad 1: MD_A01 -> /MD_AO1
- J1 pad 2: MD_A02 -> /MD_AO2
- J2 pad 1: MD_B01 -> /MD_BO1
- J2 pad 2: MD_B02 -> /MD_BO2
- J7 pad 1: /SWDIN -> /SWDIO
- U1 pad 5: GND -> Net-(U1-PH0)
- Y1 pad 1: GND -> Net-(U1-PH0)
Routing:
- net +3.3V: track 0.00 -> 221.3 mm
- net VM: track 0.00 -> 179.6 mm
- net +5V: track 0.00 -> 173.9 mm
- net Vusb: track 0.00 -> 166.7 mm, vias 0 -> 2
- net /ESD_D+: track 0.00 -> 112.2 mm, vias 0 -> 4
- net GND: track 0.00 -> 94.1 mm, vias 0 -> 57
- net /ESD_D-: track 0.00 -> 78.5 mm, vias 0 -> 4
- net /MD_PWMB: track 0.00 -> 50.6 mm
- net /WS_DIN: track 0.00 -> 39.1 mm
- net /IMU_SCL: track 0.00 -> 38.6 mm
- net /IMU_SDA: track 0.00 -> 36.9 mm
- net /IMU_INT: track 0.00 -> 35.3 mm
- net /SWDIO: track 0.00 -> 34.5 mm, vias 0 -> 2
- net /MD_BIN2: track 0.00 -> 33.4 mm
- net /MD_BIN1: track 0.00 -> 32.7 mm
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- added copper zone on B.Cu, net /ESD_D+
- added copper zone on B.Cu, net /ESD_D-
- added copper zone on B.Cu, net /SWDIO
- added copper zone on B.Cu, net GND
- added copper zone on B.Cu, net Vusb
Other:
- board text added: "Carson Giles Embedded Systems"

Commit message: Add files via upload
Parts:
- moved C14 5.63 mm to (147.5, 115.5), turned to -90 degrees
- moved D4 5.00 mm to (114.0, 112.0)
- moved F1 5.00 mm to (110.6, 118.5)
- moved J1 5.00 mm to (128.1, 112.9)
- moved J2 5.00 mm to (127.1, 124.7)
- moved J8 5.00 mm to (101.5, 126.5)
- moved R5 5.00 mm to (109.9, 123.5)
- moved R6 5.00 mm to (110.1, 130.5)
- moved R7 5.00 mm to (117.5, 125.0)
- moved R8 5.00 mm to (117.5, 128.0)
- moved R9 5.00 mm to (114.0, 114.7)
- moved U4 5.00 mm to (138.5, 116.0)
- moved U5 5.00 mm to (111.1, 126.5)
Routing:
- net Vusb: track 166.7 -> 161.7 mm
- net VM: track 179.6 -> 174.6 mm
- net /ESD_D-: track 78.5 -> 83.5 mm
- net /ESD_D+: track 112.2 -> 107.3 mm
- net /MD_PWMB: track 50.6 -> 47.6 mm
- net /MD_PWMA: track 26.8 -> 24.2 mm
- net /MD_STBY: track 31.3 -> 28.8 mm
- net +3.3V: track 221.3 -> 219.1 mm
- net /MD_AIN2: track 25.7 -> 23.7 mm
- net /MD_BIN2: track 33.4 -> 31.6 mm
- net /MD_BIN1: track 32.7 -> 30.9 mm
- net /MD_AIN1: track 25.3 -> 23.9 mm
Other:
- board outline added: 94 x 94 mm

Commit message: Add files via upload
Parts:
- C20: value 0.1 µF -> 0.01 µF
- R1, R2: value 1kΩ -> 1 kΩ
Changed lines of the file:
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@@
 		)
 		(embedded_fonts no)
-		(model "${KICAD8_3DMODEL_DIR}/Connector_PinSocket_2.54mm.3dshapes/PinSocket_2x04_P2.54mm_Vertical.wrl"
+		(model "${KICAD10_3DMODEL_DIR}/Connector_PinSocket_2.54mm.3dshapes/PinSocket_2x04_P2.54mm_Vertical.step"
 			(offset
-				(xyz 0 0 0)
+				(xyz -2.5 -7.5 0)
 			)
 			(scale
@@
 			)
 			(rotate
-				(xyz 0 0 0)
+				(xyz -0 -0 180)
+			)
+		)
+		(model "${KIPRJMOD}/components/ESP8266-01_ESP-01/step/ESP8266-01_ESP-01.step"
+			(offset
+				(xyz 8.5 -3.5 8.5)
+			)
+			(scale
+				(xyz 1 1 1)
+			)
+			(rotate
+				(xyz -90 -0 90)
 			)
 		)
@@
 			)
 		)
+		(model "${KIPRJMOD}/components/MPU6050/ITG-MPU.STEP"
+			(offset
+				(xyz -4 -29.5 5.5)
+			)
+			(scale
+				(xyz 1 1 1)
+			)
+			(rotate
+				(xyz -90 -0 180)
+			)
+		)
 	)
 	(footprint "Package_TO_SOT_SMD:SOT-223-3_TabPin2"
@@
 			)
 		)
+		(model "${KIPRJMOD}/components/LD1117S50TR_SOT223/step/LD1117S50TR.STEP"
+			(offset
+				(xyz 0 0 0)
+			)
+			(scale
+				(xyz 1 1 1)
+			)
+			(rotate
+				(xyz 90 -180 -180)
+			)
+		)
 	)
 	(footprint "Capacitor_SMD:C_0805_2012Metric_Pad1.18x1.45mm_HandSolder"
@@
 		)
 		(embedded_fonts no)
-		(model "${KICAD8_3DMODEL_DIR}/Crystal.3dshapes/Crystal_SMD_Abracon_ABM8G-4Pin_3.2x2.5mm.wrl"
+		(model "${KICAD10_3DMODEL_DIR}/Crystal.3dshapes/Crystal_SMD_Abracon_ABM8G-4Pin_3.2x2.5mm.step"
 			(offset
 				(xyz 0 0 0)
@@
 			)
 			(rotate
-				(xyz 0 0 0)
+				(xyz -0 -0 -0)
 			)
 		)
@@
 		)
 		(embedded_fonts no)
+		(model "${KIPRJMOD}/components/SPDT_Slide_Switch/step/SLW-66527511-SMT-TR.step"
+			(offset
+				(xyz 0 0 1.5)
+			)
+			(scale
+				(xyz 1 1 1)
+			)
+			(rotate
+				(xyz -90 -0 -0)
+			)
+		)
 	)
 	(footprint "Resistor_SMD:R_0805_2012Metric_Pad1.20x1.40mm_HandSolder"
@@
 			)
 		)
-		(property "Value" "1kΩ"
+		(property "Value" "1 kΩ"
 			(at 0 1.65 0)
 			(layer "F.Fab")
@@
 			)
 		)
+		(model "${KIPRJMOD}/components/LD1117S50TR_SOT223/step/LD1117S50TR.STEP"
+			(offset
+				(xyz 0 0 0)
+			)
+			(scale
+				(xyz 1 1 1)
+			)
+			(rotate
+				(xyz -90 -0 -0)
+			)
+		)
 	)
 	(footprint "Connector_PinHeader_2.54mm:PinHeader_1x04_P2.54mm_Vertical"
@@
 		)
 		(embedded_fonts no)
-		(model "${KICAD8_3DMODEL_DIR}/Connector_PinHeader_2.54mm.3dshapes/PinHeader_1x04_P2.54mm_Vertical.wrl"
+		(model "${KICAD10_3DMODEL_DIR}/Connector_PinHeader_2.54mm.3dshapes/PinHeader_1x04_P2.54mm_Vertical.step"
 			(offset
 				(xyz 0 0 0)
@@
 		)
 		(embedded_fonts no)
+		(model "${KIPRJMOD}/components/SPDT_Slide_Switch/step/SLW-66527511-SMT-TR.step"
+			(offset
+				(xyz 0 0 1.5)
+			)
+			(scale
+				(xyz 1 1 1)
+			)
+			(rotate
+				(xyz 90 180 -180)
+			)
+		)
 	)
 	(footprint "Capacitor_SMD:C_0805_2012Metric_Pad1.18x1.45mm_HandSolder"
@@
 			)
 		)
-		(property "Value" "0.1 µF"
+		(property "Value" "0.01 µF"
 			(at 0 1.68 0)
 			(layer "F.Fab")
@@
 			)
 		)
+		(model "${KIPRJMOD}/components/SW_uP_Reset/step/SW_uP_Reset.stp"
+			(offset
+				(xyz 0 0 0)
+			)
+			(scale
+				(xyz 1 1 1)
+			)
+			(rotate
+				(xyz 0 0 0)
+			)
+		)
 	)
 	(footprint "Capacitor_SMD:C_0805_2012Metric_Pad1.18x1.45mm_HandSolder"
@@
 			)
 		)
+		(model "${KIPRJMOD}/components/Stm32/step/STM32F401RBT6.STEP"
+			(offset
+				(xyz 0 0 0)
+			)
+			(scale
+				(xyz 1 1 1)
+			)
+			(rotate
+				(xyz -90 -0 -0)
+			)
+		)
 	)
 	(footprint "Capacitor_SMD:C_0805_2012Metric_Pad1.18x1.45mm_HandSolder"
@@
 			)
 		)
+		(model "${KIPRJMOD}/components/USB_C_Receptacle_USB2.0_14P/USB4105GFA060--3DModel-STEP-56544.STEP"
+			(offset
+				(xyz 0 -1 0)
+			)
+			(scale
+				(xyz 1 1 1)
+			)
+			(rotate
+				(xyz -90 -0 -0)
+			)
+		)
 	)
 	(footprint "LED_SMD:LED_0805_2012Metric_Pad1.15x1.40mm_HandSolder"
@@
 			)
 		)
+		(model "${KIPRJMOD}/components/TB6612FNG/step/TB6612FNG,C,8,EL.STEP"
+			(offset
+				(xyz 0 0 0)
+			)
+			(scale
+				(xyz 1 1 1)
+			)
+			(rotate
+				(xyz -90 -0 -0)
+			)
+		)
 	)
 	(footprint "Capacitor_SMD:C_0805_2012Metric_Pad1.18x1.45mm_HandSolder"
@@
 			)
 		)
+		(model "${KIPRJMOD}/components/Fuse_3DModel/MF-MSMF050-2--3DModel-STEP-56544.STEP"
+			(offset
+				(xyz 0 0 1)
+			)
+			(scale
+				(xyz 1 1 1)
+			)
+			(rotate
+				(xyz 90 -0 -0)
+			)
+		)
 	)
 	(footprint "Capacitor_SMD:C_0805_2012Metric_Pad1.18x1.45mm_HandSolder"
@@
 			)
 		)
+		(model "${KIPRJMOD}/components/1x4 connector/step/B4B-XH-A -LF--SN---3DModel-STEP-56544.STEP"
+			(offset
+				(xyz 3.5 -0.5 0)
+			)
+			(scale
+				(xyz 1 1 1)
+			)
+			(rotate
+				(xyz 90 -180 180)
+			)
+		)
 	)
 	(footprint "Capacitor_SMD:C_0805_2012Metric_Pad1.18x1.45mm_HandSolder"
@@
 			)
 		)
-		(property "Value" "1kΩ"
+		(property "Value" "1 kΩ"
 			(at 0 1.65 0)
 			(layer "F.Fab")
