File: BalanceRobot/kicad1.kicad_sch (KiCad schematic)
At the start: 56 parts, among them J1 M1_CONN, J2 M2_CONN, J3 BATT_CONN, J4 Conn_MPU6050, J5 ESP_CONN, J6 ENCODER_CONN, J7 Conn_01x04, J8 USB_C_Receptacle_USB2.0_14P, J9 MT6701_CONN, SW1 SW_UP_Reset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

Commit message: Add files via upload
Parts:
- C20: value 0.1 µF -> 0.01 µF
- R1, R2: value 1kΩ -> 1 kΩ
Changed lines of the file:
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@@
 			)
 		)
-		(property "Value" "0.1 µF"
+		(property "Value" "0.01 µF"
 			(at 55.626 51.562 90)
 			(show_name no)
@@
 			)
 		)
-		(property "Value" "1kΩ"
+		(property "Value" "1 kΩ"
 			(at 185.42 105.4099 0)
 			(show_name no)
@@
 			)
 		)
-		(property "Value" "1kΩ"
+		(property "Value" "1 kΩ"
 			(at 185.42 138.4299 0)
 			(show_name no)
